Commit message: 質量、モータのlimit、慣性をおおよその値で適用

File: robot_description/simple_model/simple_model.urdf (robot description, URDF)
Before this commit: robot rdc_biped_robot, 8 links, 7 joints
Links:
- link body: mass 0.1 -> 1.782
- link l_kp2heel: mass 0.1 -> 1
- link l_wp2kp: mass 0.1 -> 1
- link l_wr2wp: mass 0.1 -> 1.782
- link r_kp2heel: mass 0.1 -> 1
- link r_wp2kp: mass 0.1 -> 1
- link r_wr2wp: mass 0.1 -> 1.782
Joints:
- joint l_knee_pitch: limit lower=-1.72 upper=1.72 effort=100 velocity=100 -> lower=-6.28 upper=6.28 effort=7.2 velocity=11.519173063
- joint l_waist_pitch: limit lower=-1.72 upper=1.72 effort=100 velocity=100 -> lower=-6.28 upper=6.28 effort=7.2 velocity=11.519173063
- joint l_waist_roll: limit lower=-1.72 upper=1.72 effort=100 velocity=100 -> lower=-6.28 upper=6.28 effort=7.2 velocity=11.519173063
- joint r_knee_pitch: limit lower=-1.72 upper=1.72 effort=100 velocity=100 -> lower=-6.28 upper=6.28 effort=7.2 velocity=11.519173063
- joint r_waist_pitch: limit lower=-1.72 upper=1.72 effort=100 velocity=100 -> lower=-6.28 upper=6.28 effort=7.2 velocity=11.519173063
- joint r_waist_roll: limit lower=-1.72 upper=1.72 effort=100 velocity=100 -> lower=-6.28 upper=6.28 effort=7.2 velocity=11.519173063

Commit message: 腰リンクおよび付属ジョイントの初期高さを修正。脚が埋まる問題を解決。両足がついた状態から間島る

File: robot_description/simple_model/simple_model.urdf (robot description, URDF)
Before this commit: robot rdc_biped_robot, 8 links, 7 joints
Joints:
- joint l_waist_roll: origin xyz=0 0.105 0 rpy=0 0 0 -> xyz=0 0.105 0.364 rpy=0 0 0
- joint r_waist_roll: origin xyz=0 -0.105 0 rpy=0 0 0 -> xyz=0 -0.105 0.364 rpy=0 0 0

Commit message: 脛と足を別パーツ化

File: robot_description/simple_model/simple_model.urdf (robot description, URDF)
Before this commit: robot rdc_biped_robot, 8 links, 7 joints
Links:
- added link None, mass 0.0; collision mesh filename=meshes/stl/link_heel2end.stl scale=1 1 1; visual mesh filename=meshes/stl/link_heel2end.stl scale=1 1 1
Joints:
- added joint l_ankle: type fixed, parent l_kp2heel, child l_heel2end, origin xyz=-0.164 rpy=0 0 0
- added joint r_ankle: type fixed, parent r_kp2heel, child r_heel2end, origin xyz=-0.164 rpy=0 0 0

Commit message: Update simple_model.urdf

File: robot_description/simple_model/simple_model.urdf (robot description, URDF)
Before this commit: robot rdc_biped_robot, 9 links, 9 joints
Links:
- removed link None
- added link heel2end, mass 0.0; collision mesh filename=meshes/stl/link_heel2end.stl scale=1 1 1; visual mesh filename=meshes/stl/link_heel2end.stl scale=1 1 1
- added link r_heel2end, mass 0.0; collision mesh filename=meshes/stl/link_heel2end.stl scale=1 1 1; visual mesh filename=meshes/stl/link_heel2end.stl scale=1 1 1

Commit message: modify simple_model.urdf

File: robot_description/simple_model/simple_model.urdf (robot description, URDF)
Before this commit: robot rdc_biped_robot, 10 links, 9 joints
Links:
- removed link heel2end
- added link l_heel2end, mass 0.0; collision mesh filename=meshes/stl/link_heel2end.stl scale=1 1 1; visual mesh filename=meshes/stl/link_heel2end.stl scale=1 1 1
Joints:
- joint l_ankle: origin xyz=-0.164 rpy=0 0 0 -> xyz=0 0 -0.164 rpy=0 0 0
- joint l_waist_pitch: origin xyz=0.08 0.041 0.00 rpy=0 0 0 -> xyz=0.08 0.041 0.0 rpy=0 0 0
- joint r_ankle: origin xyz=-0.164 rpy=0 0 0 -> xyz=0 0 -0.164 rpy=0 0 0
- joint r_waist_pitch: origin xyz=0.08 -0.041 0.00 rpy=0 0 0 -> xyz=0.08 -0.041 0.0 rpy=0 0 0

Commit message: limit range of motion

File: robot_description/simple_model/simple_model.urdf (robot description, URDF)
Before this commit: robot rdc_biped_robot, 10 links, 9 joints
Links:
- link body: mass 1.782 -> 0.891
- link l_kp2heel: mass 1 -> 0.5
- link l_wp2kp: mass 1 -> 0.5
- link l_wr2wp: mass 1.782 -> 0.891
- link r_kp2heel: mass 1 -> 0.5
- link r_wp2kp: mass 1 -> 0.5
- link r_wr2wp: mass 1.782 -> 0.891
Joints:
- joint l_ankle: type fixed -> revolute
- joint l_knee_pitch: limit lower=-6.28 upper=6.28 effort=7.2 velocity=11.519173063 -> lower=-3.14 upper=-1.57 effort=7.2 velocity=11.519173063
- joint l_waist_pitch: limit lower=-6.28 upper=6.28 effort=7.2 velocity=11.519173063 -> lower=-2.35 upper=0.0 effort=7.2 velocity=11.519173063
- joint l_waist_roll: limit lower=-6.28 upper=6.28 effort=7.2 velocity=11.519173063 -> lower=-0.78 upper=0.78 effort=7.2 velocity=11.519173063
- joint r_ankle: type fixed -> revolute
- joint r_knee_pitch: limit lower=-6.28 upper=6.28 effort=7.2 velocity=11.519173063 -> lower=-3.14 upper=-1.57 effort=7.2 velocity=11.519173063
- joint r_waist_pitch: limit lower=-6.28 upper=6.28 effort=7.2 velocity=11.519173063 -> lower=-2.35 upper=0.0 effort=7.2 velocity=11.519173063
- joint r_waist_roll: limit lower=-6.28 upper=6.28 effort=7.2 velocity=11.519173063 -> lower=2.35 upper=3.92 effort=7.2 velocity=11.519173063

Commit message: update urdf

File: robot_description/simple_model/simple_model.urdf (robot description, URDF)
Before this commit: robot rdc_biped_robot, 10 links, 9 joints
Joints:
- joint l_knee_pitch: limit lower=-3.14 upper=-1.57 effort=7.2 velocity=11.519173063 -> lower=1.57 upper=4.71 effort=7.2 velocity=11.519173063
- joint l_waist_roll: limit lower=-0.78 upper=0.78 effort=7.2 velocity=11.519173063 -> lower=-3.14 upper=0 effort=7.2 velocity=11.519173063
- joint r_knee_pitch: limit lower=-3.14 upper=-1.57 effort=7.2 velocity=11.519173063 -> lower=1.57 upper=4.71 effort=7.2 velocity=11.519173063
- joint r_waist_roll: limit lower=2.35 upper=3.92 effort=7.2 velocity=11.519173063 -> lower=-3.14 upper=0 effort=7.2 velocity=11.519173063

Commit message: modifying parameters

File: robot_description/simple_model/simple_model.urdf (robot description, URDF)
Before this commit: robot rdc_biped_robot, 10 links, 9 joints
Joints:
- joint l_waist_pitch: limit lower=-2.35 upper=0.0 effort=7.2 velocity=11.519173063 -> lower=-6.28 upper=0.0 effort=7.2 velocity=11.519173063
- joint l_waist_roll: limit lower=-3.14 upper=0 effort=7.2 velocity=11.519173063 -> lower=-6.28 upper=0 effort=7.2 velocity=11.519173063
- joint r_waist_pitch: limit lower=-2.35 upper=0.0 effort=7.2 velocity=11.519173063 -> lower=-6.28 upper=0.0 effort=7.2 velocity=11.519173063
- joint r_waist_roll: limit lower=-3.14 upper=0 effort=7.2 velocity=11.519173063 -> lower=-6.28 upper=0 effort=7.2 velocity=11.519173063
