Commit message: ロボットモデルを更新。Ver1のハードとほぼ同じ寸法、質量になった。慣性も良好

File: robot_description/urdf_simple-model/simple_model.urdf (robot description, URDF)
Before this commit: robot rdc_biped_robot, 10 links, 9 joints
Links:
- added link body_luggage, mass 6.002284; collision mesh filename=meshes/stl/body_luggage.stl scale=1 1 1; visual mesh filename=meshes/stl/body_luggage.stl scale=1 1 1
- link body: mass 0.891 -> 1.128279
- link l_kp2heel: mass 0.5 -> 0.199496
- link l_wp2kp: mass 0.5 -> 0.581098
- link l_wr2wp: mass 0.891 -> 1.463019
- link r_kp2heel: mass 0.5 -> 0.199496
- link r_wp2kp: mass 0.5 -> 0.581098
- link r_wr2wp: mass 0.891 -> 1.463019
Joints:
- removed joint base_joint
- added joint CPG: type fixed, parent base_link, child body, origin xyz=0 0 0.333 rpy=0 0 0
- added joint luggage: type fixed, parent body, child body_luggage, origin xyz=-0.091 0 0 rpy=0 0 0
- joint l_ankle: origin xyz=0 0 -0.164 rpy=0 0 0 -> xyz=0 0 -0.149335 rpy=0 0 0; type revolute -> fixed
- joint l_knee_pitch: limit lower=1.57 upper=4.71 effort=7.2 velocity=11.519173063 -> lower=-6.28 upper=6.28 effort=7.2 velocity=11.519173063; origin xyz=0 0 -0.18 rpy=0 0 0 -> xyz=0 0 -0.16 rpy=0 0 0
- joint l_waist_pitch: limit lower=-6.28 upper=0.0 effort=7.2 velocity=11.519173063 -> lower=-6.28 upper=6.28 effort=7.2 velocity=11.519173063; origin xyz=0.08 0.041 0.0 rpy=0 0 0 -> xyz=0.091 0.055 0.00 rpy=0 0 0
- joint l_waist_roll: limit lower=-6.28 upper=0 effort=7.2 velocity=11.519173063 -> lower=-6.28 upper=6.28 effort=7.2 velocity=11.519173063; origin xyz=0 0.105 0.364 rpy=0 0 0 -> xyz=-0.091 0.075 0 rpy=0 0 0
- joint r_ankle: origin xyz=0 0 -0.164 rpy=0 0 0 -> xyz=0 0 -0.149335 rpy=0 0 0; type revolute -> fixed
- joint r_knee_pitch: limit lower=1.57 upper=4.71 effort=7.2 velocity=11.519173063 -> lower=-6.28 upper=6.28 effort=7.2 velocity=11.519173063; origin xyz=0 0 -0.18 rpy=0 0 0 -> xyz=0 0 -0.16 rpy=0 0 0
- joint r_waist_pitch: limit lower=-6.28 upper=0.0 effort=7.2 velocity=11.519173063 -> lower=-6.28 upper=6.28 effort=7.2 velocity=11.519173063; origin xyz=0.08 -0.041 0.0 rpy=0 0 0 -> xyz=0.091 -0.055 0.00 rpy=0 0 0
- joint r_waist_roll: limit lower=-6.28 upper=0 effort=7.2 velocity=11.519173063 -> lower=-6.28 upper=6.28 effort=7.2 velocity=11.519173063; origin xyz=0 -0.105 0.364 rpy=0 0 0 -> xyz=-0.091 -0.075 0 rpy=0 0 0
